Commit message: Gazebo simulation for visual servocontrol

File: Week2Challenge/rviz_simulation/urdf/puzzlebot_jetson_ed_urdf.urdf (robot description, URDF)
Before this commit: robot Puzzlebot Jetson-Lidar Ed., 5 links, 4 joints
Links:
- added link object; visual mesh filename=package://rviz_simulation/models/cube.stl scale=0.002 0.002 0.002
Joints:
- added joint object: type fixed, parent base_link, child object, origin xyz=0.0 0.0 50.0 rpy=0 0.0 0.0, axis 0 1 0
- joint camera_joint: origin xyz=0.045 0 0.02 -> xyz=0.1 0.0 0.04 rpy=1.57079632679 0 1.57079632679

Commit message: Implemented IBVS for reaching aruco in gazebo simulation, made corrections to camera frame rotation

File: Week2Challenge/rviz_simulation/urdf/puzzlebot_jetson_ed_urdf.urdf (robot description, URDF)
Before this commit: robot Puzzlebot Jetson-Lidar Ed., 6 links, 5 joints
Joints:
- joint camera_joint: origin xyz=0.1 0.0 0.04 rpy=1.57079632679 0 1.57079632679 -> xyz=0.1 0.0 0.04 rpy=-1.75079632679 0 -1.57079632679

Commit message: Added navigator node. Made corrections for kinematic and localisator nodes. Puzzlebot can now identify and position itself in front of selected aruco targets in visual servoing node

File: Week2Challenge/rviz_simulation/urdf/puzzlebot_jetson_ed_urdf.urdf (robot description, URDF)
Before this commit: robot Puzzlebot Jetson-Lidar Ed., 6 links, 5 joints
Links:
- removed link object
- added link aruco_box; visual mesh filename=package://rviz_simulation/models/cube.stl scale=0.0025 0.0025 0.0025
Joints:
- removed joint object
- added joint aruco_joint: type fixed, parent base_link, child aruco_box, origin xyz=0.0 0.0 50.0 rpy=0.0 0.0 0.0, axis 0 1 0
- joint camera_joint: origin xyz=0.1 0.0 0.04 rpy=-1.75079632679 0 -1.57079632679 -> xyz=0.1 0.0 0.04 rpy=-1.57079632679 0 -1.57079632679

Commit message: Updates: grid map

File: Week2Challenge/rviz_simulation/urdf/puzzlebot_jetson_ed_urdf.urdf (robot description, URDF)
Before this commit: robot Puzzlebot Jetson-Lidar Ed., 6 links, 5 joints
Links:
- removed link aruco_box
- added link lidar_link
Joints:
- removed joint aruco_joint
- added joint lidar_joint: type fixed, parent chassis, child lidar_link, origin xyz=0.05 0.0 0.08 rpy=0 0 0
